Commit message: Runs both the controller and sim from one launch file

File: src/arm_controller/urdf/arm_cad.urdf.xacro (robot description, xacro)
@@ -26,18 +26,18 @@
       <origin xyz="0 0 0" rpy="0 0 0" />
       <geometry>
-        <mesh filename="package://arm_sim/meshes/base_link.stl" scale="0.001 0.001 0.001" />
-      </geometry>
-      <material name="grey" />
-    </visual>
-  <collision><origin xyz="0 0 0" rpy="0 0 0" /><geometry><mesh filename="package://arm_sim/meshes/base_link.stl" scale="0.000980 0.000980 0.000980" /></geometry></collision><inertial><origin xyz="0.056552 0.012384 -0.025918" rpy="0 0 0" /><mass value="2.701002" /><inertia ixx="0.007655" ixy="-0.001141" ixz="0.0001262" iyy="0.00284" iyz="0.0001269" izz="0.007935" /></inertial></link>
+        <mesh filename="package://arm_controller/meshes/base_link.stl" scale="0.001 0.001 0.001" />
+      </geometry>
+      <material name="grey" />
+    </visual>
+  <collision><origin xyz="0 0 0" rpy="0 0 0" /><geometry><mesh filename="package://arm_controller/meshes/base_link.stl" scale="0.000980 0.000980 0.000980" /></geometry></collision><inertial><origin xyz="0.056552 0.012384 -0.025918" rpy="0 0 0" /><mass value="2.701002" /><inertia ixx="0.007655" ixy="-0.001141" ixz="0.0001262" iyy="0.00284" iyz="0.0001269" izz="0.007935" /></inertial></link>
   <link name="base_plate">
     <visual>
       <origin xyz="0 0 0" rpy="0 0 0" />
       <geometry>
-        <mesh filename="package://arm_sim/meshes/base_plate.stl" scale="0.001 0.001 0.001" />
-      </geometry>
-      <material name="grey" />
-    </visual>
-  <collision><origin xyz="0 0 0" rpy="0 0 0" /><geometry><mesh filename="package://arm_sim/meshes/base_plate.stl" scale="0.000980 0.000980 0.000980" /></geometry></collision><inertial><origin xyz="0.042843 0.029280 -0.008767" rpy="0 0 0" /><mass value="2.251151" /><inertia ixx="0.007401" ixy="0.000012823" ixz="0.000000032" iyy="0.009356" iyz="0.000003011" izz="0.016740" /></inertial></link>
+        <mesh filename="package://arm_controller/meshes/base_plate.stl" scale="0.001 0.001 0.001" />
+      </geometry>
+      <material name="grey" />
+    </visual>
+  <collision><origin xyz="0 0 0" rpy="0 0 0" /><geometry><mesh filename="package://arm_controller/meshes/base_plate.stl" scale="0.000980 0.000980 0.000980" /></geometry></collision><inertial><origin xyz="0.042843 0.029280 -0.008767" rpy="0 0 0" /><mass value="2.251151" /><inertia ixx="0.007401" ixy="0.000012823" ixz="0.000000032" iyy="0.009356" iyz="0.000003011" izz="0.016740" /></inertial></link>
   <joint name="base_joint" type="fixed">
     <parent link="base_link" />
@@ -56,18 +56,18 @@
       <origin xyz="0.059 0 0" rpy="0 1.57 0" />
       <geometry>
-        <mesh filename="package://arm_sim/meshes/shoulder_link.stl" scale="0.001 0.001 0.001" />
-      </geometry>
-      <material name="grey" />
-    </visual>
-  <collision><origin xyz="0.059 0 0" rpy="0 1.57 0" /><geometry><mesh filename="package://arm_sim/meshes/shoulder_link.stl" scale="0.000980 0.000980 0.000980" /></geometry></collision><inertial><origin xyz="-0.013715 0.000019 0.029138" rpy="0 0 0" /><mass value="3.428008" /><inertia ixx="0.02524" ixy="2.94448e-7" ixz="-0.004523" iyy="0.02879" iyz="-1.6458e-6" izz="0.006357" /></inertial></link>
+        <mesh filename="package://arm_controller/meshes/shoulder_link.stl" scale="0.001 0.001 0.001" />
+      </geometry>
+      <material name="grey" />
+    </visual>
+  <collision><origin xyz="0.059 0 0" rpy="0 1.57 0" /><geometry><mesh filename="package://arm_controller/meshes/shoulder_link.stl" scale="0.000980 0.000980 0.000980" /></geometry></collision><inertial><origin xyz="-0.013715 0.000019 0.029138" rpy="0 0 0" /><mass value="3.428008" /><inertia ixx="0.02524" ixy="2.94448e-7" ixz="-0.004523" iyy="0.02879" iyz="-1.6458e-6" izz="0.006357" /></inertial></link>
   <link name="shoulder_plate">
     <visual>
       <origin xyz="-0.043511 0.012448 -0.03425" rpy="0 0 0" />
       <geometry>
-        <mesh filename="package://arm_sim/meshes/shoulder_plate.stl" scale="0.001 0.001 0.001" />
-      </geometry>
-      <material name="grey" />
-    </visual>
-  <collision><origin xyz="-0.043511 0.012448 -0.03425" rpy="0 0 0" /><geometry><mesh filename="package://arm_sim/meshes/shoulder_plate.stl" scale="0.000980 0.000980 0.000980" /></geometry></collision><inertial><origin xyz="-0.000183 0.000000 -0.002000" rpy="0 0 0" /><mass value="1.238335" /><inertia ixx="0.004587" ixy="0" ixz="0" iyy="0.003748" iyz="0" izz="0.008332" /></inertial></link>
+        <mesh filename="package://arm_controller/meshes/shoulder_plate.stl" scale="0.001 0.001 0.001" />
+      </geometry>
+      <material name="grey" />
+    </visual>
+  <collision><origin xyz="-0.043511 0.012448 -0.03425" rpy="0 0 0" /><geometry><mesh filename="package://arm_controller/meshes/shoulder_plate.stl" scale="0.000980 0.000980 0.000980" /></geometry></collision><inertial><origin xyz="-0.000183 0.000000 -0.002000" rpy="0 0 0" /><mass value="1.238335" /><inertia ixx="0.004587" ixy="0" ixz="0" iyy="0.003748" iyz="0" izz="0.008332" /></inertial></link>
   <joint name="shoulder_fixed_joint" type="fixed">
     <parent link="shoulder_plate" />
@@ -79,9 +79,9 @@
       <origin xyz="0 0 0" rpy="0 1.57 0" />
       <geometry>
-        <mesh filename="package://arm_sim/meshes/shoulder_fixed_link.stl" scale="0.001 0.001 0.001" />
-      </geometry>
-      <material name="grey" />
-    </visual>
-  <collision><origin xyz="0 0 0" rpy="0 1.57 0" /><geometry><mesh filename="package://arm_sim/meshes/shoulder_fixed_link.stl" scale="0.000980 0.000980 0.000980" /></geometry></collision><inertial><origin xyz="-0.016486 0.000000 -0.035108" rpy="0 0 0" /><mass value="1.059660" /><inertia ixx="0.00265" ixy="0" ixz="6.3793e-05" iyy="0.001397" iyz="0" izz="0.001396" /></inertial></link>
+        <mesh filename="package://arm_controller/meshes/shoulder_fixed_link.stl" scale="0.001 0.001 0.001" />
+      </geometry>
+      <material name="grey" />
+    </visual>
+  <collision><origin xyz="0 0 0" rpy="0 1.57 0" /><geometry><mesh filename="package://arm_controller/meshes/shoulder_fixed_link.stl" scale="0.000980 0.000980 0.000980" /></geometry></collision><inertial><origin xyz="-0.016486 0.000000 -0.035108" rpy="0 0 0" /><mass value="1.059660" /><inertia ixx="0.00265" ixy="0" ixz="6.3793e-05" iyy="0.001397" iyz="0" izz="0.001396" /></inertial></link>
   <joint name="shoulder_joint" type="revolute">
     <parent link="shoulder_fixed_link" />
@@ -95,9 +95,9 @@
       <origin xyz="0.0095 0.000037 0.000028" rpy="0 1.57 0" />
       <geometry>
-        <mesh filename="package://arm_sim/meshes/elbow_fixed_link.stl" scale="0.001 0.001 0.001" />
-      </geometry>
-      <material name="grey" />
-    </visual>
-  <collision><origin xyz="0.0095 0.000037 0.000028" rpy="0 1.57 0" /><geometry><mesh filename="package://arm_sim/meshes/elbow_fixed_link.stl" scale="0.000980 0.000980 0.000980" /></geometry></collision><inertial><origin xyz="-0.062352 0.000033 -0.022604" rpy="0 0 0" /><mass value="2.997488" /><inertia ixx="0.006981" ixy="0" ixz="-0.0003831" iyy="0.005413" iyz="0" izz="0.002412" /></inertial></link>
+        <mesh filename="package://arm_controller/meshes/elbow_fixed_link.stl" scale="0.001 0.001 0.001" />
+      </geometry>
+      <material name="grey" />
+    </visual>
+  <collision><origin xyz="0.0095 0.000037 0.000028" rpy="0 1.57 0" /><geometry><mesh filename="package://arm_controller/meshes/elbow_fixed_link.stl" scale="0.000980 0.000980 0.000980" /></geometry></collision><inertial><origin xyz="-0.062352 0.000033 -0.022604" rpy="0 0 0" /><mass value="2.997488" /><inertia ixx="0.006981" ixy="0" ixz="-0.0003831" iyy="0.005413" iyz="0" izz="0.002412" /></inertial></link>
   <joint name="elbow_fixed_joint" type="fixed">
     <parent link="shoulder_link" />
@@ -109,12 +109,13 @@
       <origin xyz="0.05650 0.000015 -0.000011" rpy="0 1.57 0" />
       <geometry>
-        <mesh filename="package://arm_sim/meshes/elbow_link.stl" scale="0.001 0.001 0.001" />
-      </geometry>
-      <material name="grey" />
-    </visual>
-  <collision><origin xyz="0.05650 0.000015 -0.000011" rpy="0 1.57 0" /><geometry><mesh filename="package://arm_sim/meshes/elbow_link.stl" scale="0.000980 0.000980 0.000980" /></geometry></collision><inertial><origin xyz="-0.004749 -0.020998 -0.009823" rpy="0 0 0" /><mass value="4.315948" /><inertia ixx="0.02688" ixy="-0.004865" ixz="-0.002265" iyy="0.01063" iyz="-0.008816" izz="0.02543" /></inertial></link>
+        <mesh filename="package://arm_controller/meshes/elbow_link.stl" scale="0.001 0.001 0.001" />
+      </geometry>
+      <material name="grey" />
+    </visual>
+  <collision><origin xyz="0.05650 0.000015 -0.000011" rpy="0 1.57 0" /><geometry><mesh filename="package://arm_controller/meshes/elbow_link.stl" scale="0.000980 0.000980 0.000980" /></geometry></collision><inertial><origin xyz="-0.004749 -0.020998 -0.009823" rpy="0 0 0" /><mass value="4.315948" /><inertia ixx="0.02688" ixy="-0.004865" ixz="-0.002265" iyy="0.01063" iyz="-0.008816" izz="0.02543" /></inertial></link>
   <joint name="elbow_joint" type="revolute">
     <parent link="elbow_fixed_link" />
     <child link="elbow_link" />
+    <!-- rpy aligns Link 2 (forearm) collinearly with Link 1 (upper arm) at elbow=0 -->
     <origin xyz="-0.047 0.000022 0.000039" rpy="-2.00719 0 0" />
     <axis xyz="1 0 0" />
@@ -125,9 +126,9 @@
       <origin xyz="0.053 -0.11750 -0.051802" rpy="0 -0.43633 1.57" />
       <geometry>
-        <mesh filename="package://arm_sim/meshes/bevel_link.stl" scale="0.001 0.001 0.001" />
+        <mesh filename="package://arm_controller/meshes/bevel_link.stl" scale="0.001 0.001 0.001" />
       </geometry>
       <material name="dark_grey" />
     </visual>
-  <collision><origin xyz="0.053 -0.11750 -0.051802" rpy="0 -0.43633 1.57" /><geometry><mesh filename="package://arm_sim/meshes/bevel_link.stl" scale="0.000980 0.000980 0.000980" /></geometry></collision><inertial><origin xyz="-0.061635 -0.088296 -0.038857" rpy="0 0 0" /><mass value="12.003086" /><inertia ixx="0.05331" ixy="-0.001329" ixz="0.001766" iyy="0.1777" iyz="-0.01317" izz="0.2008" /></inertial></link>
+  <collision><origin xyz="0.053 -0.11750 -0.051802" rpy="0 -0.43633 1.57" /><geometry><mesh filename="package://arm_controller/meshes/bevel_link.stl" scale="0.000980 0.000980 0.000980" /></geometry></collision><inertial><origin xyz="-0.061635 -0.088296 -0.038857" rpy="0 0 0" /><mass value="12.003086" /><inertia ixx="0.05331" ixy="-0.001329" ixz="0.001766" iyy="0.1777" iyz="-0.01317" izz="0.2008" /></inertial></link>
   <joint name="elbow_bevel_joint" type="fixed">
     <parent link="elbow_link" />
@@ -155,9 +156,9 @@
       <origin xyz="0.05300 -0.000208 0.002892" rpy="0 -0.43633 1.57" />
       <geometry>
-        <mesh filename="package://arm_sim/meshes/wrist_pitch_link.stl" scale="0.001 0.001 0.001" />
+        <mesh filename="package://arm_controller/meshes/wrist_pitch_link.stl" scale="0.001 0.001 0.001" />
       </geometry>
       <material name="dark_grey" />
     </visual>
-  <collision><origin xyz="0.05300 -0.000208 0.002892" rpy="0 -0.43633 1.57" /><geometry><mesh filename="package://arm_sim/meshes/wrist_pitch_link.stl" scale="0.000980 0.000980 0.000980" /></geometry></collision><inertial><origin xyz="-0.063524 -0.035498 -0.017454" rpy="0 0 0" /><mass value="2.209229" /><inertia ixx="0.005389" ixy="0.0001799" ixz="8.496e-05" iyy="0.003108" iyz="-0.001965" izz="0.005901" /></inertial></link>
+  <collision><origin xyz="0.05300 -0.000208 0.002892" rpy="0 -0.43633 1.57" /><geometry><mesh filename="package://arm_controller/meshes/wrist_pitch_link.stl" scale="0.000980 0.000980 0.000980" /></geometry></collision><inertial><origin xyz="-0.063524 -0.035498 -0.017454" rpy="0 0 0" /><mass value="2.209229" /><inertia ixx="0.005389" ixy="0.0001799" ixz="8.496e-05" iyy="0.003108" iyz="-0.001965" izz="0.005901" /></inertial></link>
   <joint name="wrist_roll_joint" type="revolute">
     <parent link="wrist_pitch_link" />
@@ -178,9 +179,9 @@
       <origin xyz="-0.025013 0.115386 0.022301" rpy="0 0 0" />
       <geometry>
-        <mesh filename="package://arm_sim/meshes/gripper_link.stl" scale="0.001 0.001 0.001" />
+        <mesh filename="package://arm_controller/meshes/gripper_link.stl" scale="0.001 0.001 0.001" />
       </geometry>
       <material name="orange" />
     </visual>
-  <collision><origin xyz="-0.025013 0.115386 0.022301" rpy="0 0 0" /><geometry><mesh filename="package://arm_sim/meshes/gripper_link.stl" scale="0.000980 0.000980 0.000980" /></geometry></collision><inertial><origin xyz="-0.059103 -0.069608 -0.070075" rpy="0 0 0" /><mass value="2.237313" /><inertia ixx="0.006089" ixy="0" ixz="0" iyy="0.002719" iyz="-0.002466" izz="0.005166" /></inertial></link>
+  <collision><origin xyz="-0.025013 0.115386 0.022301" rpy="0 0 0" /><geometry><mesh filename="package://arm_controller/meshes/gripper_link.stl" scale="0.000980 0.000980 0.000980" /></geometry></collision><inertial><origin xyz="-0.059103 -0.069608 -0.070075" rpy="0 0 0" /><mass value="2.237313" /><inertia ixx="0.006089" ixy="0" ixz="0" iyy="0.002719" iyz="-0.002466" izz="0.005166" /></inertial></link>
   <joint name="gripper_joint" type="revolute">
     <parent link="gripper_link" />
@@ -202,9 +203,9 @@
       <origin xyz="-0.024892 0.05096 0.0066" rpy="0 0 0" />
       <geometry>
-        <mesh filename="package://arm_sim/meshes/upper_jaw_link.stl" scale="0.001 0.001 0.001" />
+        <mesh filename="package://arm_controller/meshes/upper_jaw_link.stl" scale="0.001 0.001 0.001" />
       </geometry>
       <material name="orange" />
     </visual>
-  <collision><origin xyz="-0.024892 0.05096 0.0066" rpy="0 0 0" /><geometry><mesh filename="package://arm_sim/meshes/upper_jaw_link.stl" scale="0.000980 0.000980 0.000980" /></geometry></collision><inertial><origin xyz="-0.059030 -0.189641 -0.083641" rpy="0 0 0" /><mass value="0.770764" /><inertia ixx="0.0008414" ixy="0.0" ixz="0.0" iyy="0.000538" iyz="-0.0002905" izz="0.001075" /></inertial></link>
+  <collision><origin xyz="-0.024892 0.05096 0.0066" rpy="0 0 0" /><geometry><mesh filename="package://arm_controller/meshes/upper_jaw_link.stl" scale="0.000980 0.000980 0.000980" /></geometry></collision><inertial><origin xyz="-0.059030 -0.189641 -0.083641" rpy="0 0 0" /><mass value="0.770764" /><inertia ixx="0.0008414" ixy="0.0" ixz="0.0" iyy="0.000538" iyz="-0.0002905" izz="0.001075" /></inertial></link>
 <!-- ========================= -->
 <!-- ros2_control -->
@@ -255,5 +256,4 @@
   </joint>
 </ros2_control>
-<!--ROS GAZEBO INTEGRATION PLUGIN -->
 <gazebo>
   <plugin
@@ -261,5 +261,5 @@
       name="gz_ros2_control::GazeboSimROS2ControlPlugin">
     <parameters>
-      $(find arm_sim)/config/ros2_controllers.yaml
+      $(find arm_controller)/config/ros2_controllers.yaml
     </parameters>
   </plugin>
