Commit message: Added Camera simuulation to arm_sim

File: src/arm_sim/urdf/arm_cad.urdf.xacro (robot description, xacro)
@@ -1,4 +1,5 @@
 <?xml version="1.0"?>
 <robot xmlns:xacro="http://www.ros.org/wiki/xacro" name="arm">
+<xacro:include filename="$(find realsense2_description)/urdf/_d435i.urdf.xacro"/>
 <xacro:arg name="use_mock_hardware" default="false"/>
 <xacro:arg name="use_gazebo" default="false"/>
@@ -198,4 +199,15 @@
   </joint>
   <link name="tool0"/>
+  <!-- ========================= -->
+  <!-- Intel RealSense D435i -->
+  <!-- ========================= -->
+  <xacro:sensor_d435i
+    parent="gripper_link"
+    name="camera"
+    use_nominal_extrinsics="true">
+    <origin
+        xyz="0 0.03 0.07"
+        rpy="0 0 ${PI/2}"/>
+  </xacro:sensor_d435i>
   <link name="upper_jaw_link">
     <visual>
@@ -265,4 +277,29 @@
   </plugin>
 </gazebo>
+<!-- ========================= -->
+<!-- D435i Gazebo RGB-D sensor -->
+<!-- ========================= -->
+<gazebo reference="camera_link">
+  <sensor name="d435i_rgbd" type="rgbd_camera">
+    <always_on>true</always_on>
+    <visualize>true</visualize>
+    <update_rate>30</update_rate>
+    <topic>camera</topic>
+    <gz_frame_id>camera_link</gz_frame_id>
+    <camera>
+      <horizontal_fov>1.211</horizontal_fov>
+      <camera_info_topic>camera/camera_info</camera_info_topic>
+      <image>
+        <width>1920</width>
+        <height>1080</height>
+        <format>R8G8B8</format>
+      </image>
+      <clip>
+        <near>0.1</near>
+        <far>10.0</far>
+      </clip>
+    </camera>
+  </sensor>
+</gazebo>
 <!--Camera Part Removed -->
 </robot>

Commit message: Added Camera Sensors. Made a Dashboard for the Camera. Fixed the RTF using not loading gazebo.

File: src/arm_sim/urdf/arm_cad.urdf.xacro (robot description, xacro)
@@ -17,4 +17,7 @@
     <color rgba="0 0 0 0" />
   </material>
+  <material name="red">
+    <color rgba="1.0 0.0 0.0 1.0" />
+  </material>
   <link name="world" />
   <joint name="world_to_base" type="fixed">
@@ -210,4 +213,38 @@
         rpy="0 0 ${PI/2}"/>
   </xacro:sensor_d435i>
+  <!-- ========================= -->
+  <!-- Elbow camera (sensor only) -->
+  <!-- ========================= -->
+  <link name="elbow_camera_link">
+    <visual>
+      <origin xyz="0 0 0" rpy="0 0 0" />
+      <geometry>
+        <box size="0.02 0.02 0.005" />
+      </geometry>
+      <material name="red" />
+    </visual>
+  </link>
+  <joint name="elbow_camera_joint" type="fixed">
+    <parent link="elbow_link"/>
+    <child link="elbow_camera_link"/>
+    <origin xyz="-0.06 0 0.05" rpy="0 0.4363 ${-PI/2}"/>
+  </joint>
+  <!-- ========================= -->
+  <!-- Gripper Camera (sensor only) -->
+  <!-- ========================= -->
+  <link name="gripper_camera_link">
+    <visual>
+      <origin xyz="0 0 0" rpy="0 0 0" />
+      <geometry>
+        <box size="0.001 0.015 0.015" />
+      </geometry>
+      <material name="red" />
+    </visual>
+  </link>
+  <joint name="gripper_camera_joint" type="fixed">
+    <parent link="gripper_link"/>
+    <child link="gripper_camera_link"/>
+    <origin xyz="0 0.105 0" rpy="0 0 ${PI/2}"/>
+  </joint>
   <link name="upper_jaw_link">
     <visual>
@@ -291,6 +328,6 @@
       <camera_info_topic>camera/camera_info</camera_info_topic>
       <image>
-        <width>1920</width>
-        <height>1080</height>
+        <width>640</width>
+        <height>480</height>
         <format>R8G8B8</format>
       </image>
@@ -302,4 +339,48 @@
   </sensor>
 </gazebo>
+<gazebo reference="elbow_camera_link">
+  <sensor name="elbow_camera" type="camera">
+    <always_on>true</always_on>
+    <visualize>true</visualize>
+    <update_rate>30</update_rate>
+    <topic>elbow_camera/image</topic>
+    <gz_frame_id>elbow_camera_link</gz_frame_id>
+    <camera>
+      <horizontal_fov>1.047</horizontal_fov>
+      <camera_info_topic>elbow_camera/camera_info</camera_info_topic>
+      <image>
+        <width>640</width>
+        <height>480</height>
+        <format>R8G8B8</format>
+      </image>
+      <clip>
+        <near>0.05</near>
+        <far>10.0</far>
+      </clip>
+    </camera>
+  </sensor>
+</gazebo>
+<gazebo reference="gripper_camera_link">
+  <sensor name="gripper_camera" type="camera">
+    <always_on>true</always_on>
+    <visualize>true</visualize>
+    <update_rate>30</update_rate>
+    <topic>gripper_camera/image</topic>
+    <gz_frame_id>gripper_camera_link</gz_frame_id>
+    <camera>
+      <horizontal_fov>1.047</horizontal_fov>
+      <camera_info_topic>gripper_camera/camera_info</camera_info_topic>
+      <image>
+        <width>640</width>
+        <height>480</height>
+        <format>R8G8B8</format>
+      </image>
+      <clip>
+        <near>0.05</near>
+        <far>10.0</far>
+      </clip>
+    </camera>
+  </sensor>
+</gazebo>
 <!--Camera Part Removed -->
 </robot>
